File: Controller.kicad_sch (KiCad schematic)
At the start: 91 parts, among them J1 Conn_01x03, J2 Conn_02x05_Odd_Even, J4 770669-5, Q1 MMBT3904, U1 VX7803-500, U10 LMV358IDGKR, U11 TPS1HB16-Q1, U12 CL220K4-G, U13 CL220K4-G, U14 PC357, U15 PC357, U16 CL220K4-G, U17 CL220K4-G, U18 PC357, U19 PC357, U2 VX7805-500, U3 STM32F412RGTx, U4 LSM6DS3, U5 MCP2561-E-P, U6 TPS1HB16-Q1, U7 M12D-04PMMR-SF7003, U8 PCF85063AT/AAZ, U9 LMV358IDGKR, Y1 X32K768S301

Commit message: includingImages
Other:
- note added: "Grounded Mounts and Indicator LEDS"
- note added: "High Side Drivers"
- note added: "Powersupply allows for variable voltage input up to 32V and protection for Alternator Load Dump"
- note added: "Raspberry Pi Compute Unit 4"
- note added: "STM32 Microcontroller"
- note removed: "Add delayed startup and undervoltage lockout?"
- note removed: "Do I need to change the feedback pin?"
- note removed: "Still need to workout startup and shutdown logic"
- moved on the sheet: C10, C11, C12, C13, C14, C15, C20, C22, C24, C25, C5, C6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
